File: Nandy/nandy.kicad_pcb (KiCad board)
At the start: 2 copper layers, 30.5 x 25.4 mm, 9 parts, among them Q1 Q_NPN_CBE, Q2 Q_NPN_CBE

Commit message: add logo and website link
Parts:
- added Ref**: Val**, random stuff:mothface, B.Cu at (156.2, 66.2)
Other:
- board text added: "moth.monster"

Commit message: total redesign
Parts:
- removed 1: Input 2, Connector_PinHeader_2.54mm:PinHeader_1x01_P2.54mm_Vertical
- removed 1kΩ: 200, Resistor_THT:R_Axial_DIN0207_L6.3mm_D2.5mm_P7.62mm_Horizontal
- removed 2: Input 1, Connector_PinHeader_2.54mm:PinHeader_1x01_P2.54mm_Vertical
- removed 5V: 5V, Connector_PinHeader_2.54mm:PinHeader_1x01_P2.54mm_Vertical
- removed GND: GND, Connector_PinHeader_2.54mm:PinHeader_1x01_P2.54mm_Vertical
- removed OUT: Output, Connector_PinHeader_2.54mm:PinHeader_1x01_P2.54mm_Vertical
- removed Q1, Q2: Q_NPN_CBE, Package_TO_SOT_THT:TO-92
- removed the REF** at (156.8, 58.4)
- removed the Ref** at (156.2, 66.2)
- added J1: Conn_01x02, Connector_PinHeader_2.54mm:PinHeader_1x02_P2.54mm_Vertical, B.Cu at (83.8, 129.5)
- added J2: Conn_01x02, Connector_PinHeader_2.54mm:PinHeader_1x02_P2.54mm_Vertical, B.Cu at (83.8, 121.9)
- added J4: OUT, Connector_PinHeader_2.54mm:PinHeader_1x01_P2.54mm_Vertical, B.Cu at (96.5, 127.0)
- added REF**: OSHW-Symbol_8.9x8mm_Copper, Symbol:OSHW-Symbol_8.9x8mm_Copper, F.Cu at (88.9, 127.0)
- added Ref**: Val**, random stuff:mothfacefixed, B.Cu at (90.8, 123.2)
- added U1: 74LVC2G00, Package_SO:VSSOP-8_2.3x2mm_P0.5mm, B.Cu at (88.9, 127.0)
Routing:
- net Net-(J5-Pad1): track 18.7 -> 0.00 mm
- net Net-(J2-Pad1): track 12.2 -> 0.00 mm
- net GND: track 0.00 -> 11.0 mm
- net Net-(J3-Pad1): track 8.67 -> 0.00 mm
- net VCC: track 0.00 -> 8.42 mm
- net Net-(J1-Pad1): track 12.2 -> 4.27 mm
- net Net-(J4-Pad1): track 13.5 -> 6.17 mm
- net Net-(Q1-Pad3): track 6.35 -> 0.00 mm
- net Net-(J2-Pad2): track 0.00 -> 4.69 mm
Other:
- board size 30.5 x 25.4 mm -> 17.7 x 15.2 mm
- rule pad_to_mask_clearance: 0.05 -> 0
- board text added: "+"
- board text added: "-"
- board text added: "1"
- board text added: "2"
- board text added: "OUT"
- board text added: "made by eri CC-BY-SA"
- board text removed: "CC-BY-SA"
- board text removed: "made by eri"
- board text removed: "moth.monster"

Commit message: Add files via upload
Parts:
- removed Ref**: Val**, random stuff:mothfacefixed
