File: nandy/nandy.kicad_pcb (KiCad board)
At the start: 2 copper layers, 14 x 16.5 mm, 5 parts, among them J1 Conn_01x02_Male, J2 Conn_01x02_Male, J3 OUT, U1 74LVC1G00

Commit message: Add files via upload
Parts:
- removed G***: LOGO, mothface:mothfacesmoler
